File: HardWare/V1_ robot_controller/V1_ robot_controller.kicad_sch (KiCad schematic)
At the start: 27 parts, among them J1 XT30UPB-M, J10 Conn_01x05_Pin, J11 Conn_01x05_Pin, J12 Conn_01x05_Pin, J13 Conn_01x05_Pin, J14 Conn_01x03_Pin, J2 XT30UPB-M, J3 Conn_01x02_Pin, J4 Conn_01x02_Pin, J6 Conn_01x03_Pin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

Commit message: m,
jkgh
Parts:
- removed C4: 220uf / 25v, Capacitor_THT:CP_Radial_D8.0mm_P3.80mm, symbol Device:C_Polarized
- removed J10, J11, J12, J13, J8, J9: Conn_01x05_Pin, Connector_PinHeader_2.54mm:PinHeader_1x05_P2.54mm_Vertical, symbol Connector:Conn_01x05_Pin
- removed R1, R2: 10k, Resistor_SMD:R_0805_2012Metric_Pad1.20x1.40mm_HandSolder, symbol Device:R
- removed U4: PCF8574AT, Package_SO:SOIC-16W_7.5x10.3mm_P1.27mm, symbol Interface_Expansion:PCF8574AT
- removed U5: LEVEL-SHIFTER-4ch, BOB-12009:CONV_BOB-12009, symbol BOB-12009:BOB-12009
- added C5: 220uf / 25v, Capacitor_THT:CP_Radial_D6.3mm_P2.50mm, symbol Device:C_Polarized
- added J10, J11, J12, J13, J5, J8, J9: Conn_01x04_Pin, Connector_PinHeader_2.54mm:PinHeader_1x04_P2.54mm_Vertical, symbol Connector:Conn_01x04_Pin
- added SW3: SW_Push, Button_Switch_THT:SW_PUSH_6mm_H4.3mm, symbol Switch:SW_Push
- added U4: BOB-12009, BOB-12009:CONV_BOB-12009, symbol BOB-12009:BOB-12009
Connections:
- net +3.3V: now also J10.1 (Pin_1), J11.1 (Pin_1), J12.1 (Pin_1), J13.1 (Pin_1), J5.1 (Pin_1), J8.1 (Pin_1), J9.1 (Pin_1), U4.LV
- net +5V: now also C5.1, U4.HV
- net GND: now also C5.2, J10.2 (Pin_2), J11.2 (Pin_2), J12.2 (Pin_2), J13.2 (Pin_2), J5.2 (Pin_2), J8.2 (Pin_2), J9.2 (Pin_2), SW3.1, U4.GND_1 (GND), U4.GND_2 (GND)
- net QTR_DER: now also U4.LV1
- net QTR_IZQ: now also U4.LV2
- net SCL: now also J10.3 (Pin_3), J11.3 (Pin_3), J12.3 (Pin_3), J13.3 (Pin_3), J5.4 (Pin_4), J8.3 (Pin_3), J9.3 (Pin_3)
- net SDA: now also J10.4 (Pin_4), J11.4 (Pin_4), J12.4 (Pin_4), J13.4 (Pin_4), J5.3 (Pin_3), J8.4 (Pin_4), J9.4 (Pin_4)
- net at U3.4 (A01): now also J4.1 (Pin_1); no longer J4.2 (Pin_2)
- net at U3.5 (A02): now also J4.2 (Pin_2); no longer J4.1 (Pin_1)
- net at J14.3 (Pin_3): now also U1.2 (GPIO2); no longer U1.1 (GPIO1)
- net at J6.3 (Pin_3): now also U4.HV1
- net at J7.3 (Pin_3): now also U4.HV2
- new net: SW3.2, U1.1 (GPIO1)
- no-connect marks 6 -> 1
Other:
- moved on the sheet: J4, SW2
