File: HardWare/V1_ robot_controller/V1_ robot_controller.kicad_pcb (KiCad board)
At the start: 2 copper layers, 19 parts, among them J1 XT30UPB-M, J2 XT30UPB-M, J3 Conn_01x02_Pin, J4 Conn_01x02_Pin, J5 Conn_01x02_Pin, SW1 SW_SPDT, SW2 SW_Push, U1 ESP32-C3_SUPERMINI_TH, U2 L7805, U3 TB6612 FNG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

Commit message: kicad
empece el diseño en kicad
Parts:
- removed J5: Conn_01x02_Pin, Connector_PinHeader_2.54mm:PinHeader_1x02_P2.54mm_Vertical
- added J10: Conn_01x05_Pin, Connector_PinHeader_2.54mm:PinHeader_1x05_P2.54mm_Vertical, F.Cu at (149.4, 23.8)
- added J11: Conn_01x05_Pin, Connector_PinHeader_2.54mm:PinHeader_1x05_P2.54mm_Vertical, F.Cu at (144.7, 23.8)
- added J12: Conn_01x05_Pin, Connector_PinHeader_2.54mm:PinHeader_1x05_P2.54mm_Vertical, F.Cu at (163.3, 23.8)
- added J13: Conn_01x05_Pin, Connector_PinHeader_2.54mm:PinHeader_1x05_P2.54mm_Vertical, F.Cu at (168.0, 23.8)
- added J14: Conn_01x03_Pin, Connector_PinHeader_2.54mm:PinHeader_1x03_P2.54mm_Vertical, F.Cu at (129.6, 44.5)
- added J6: Conn_01x03_Pin, Connector_PinHeader_2.54mm:PinHeader_1x03_P2.54mm_Vertical, F.Cu at (140.8, 28.8)
- added J7: Conn_01x03_Pin, Connector_PinHeader_2.54mm:PinHeader_1x03_P2.54mm_Vertical, F.Cu at (137.0, 28.9)
- added J8: Conn_01x05_Pin, Connector_PinHeader_2.54mm:PinHeader_1x05_P2.54mm_Vertical, F.Cu at (158.7, 23.8)
- added J9: Conn_01x05_Pin, Connector_PinHeader_2.54mm:PinHeader_1x05_P2.54mm_Vertical, F.Cu at (154.0, 23.8)
- C3: footprint Capacitor_THT:CP_Radial_D8.0mm_P3.80mm -> Capacitor_THT:CP_Radial_D6.3mm_P2.50mm
- U2: footprint Package_TO_SOT_THT:TO-220-3_Vertical -> Package_TO_SOT_THT:TO-220F-3_Horizontal_TabUp
- moved D1 152.2 mm to (195.0, 42.3), turned to 90 degrees
- moved J2 151.8 mm to (202.0, 42.2)
- moved J1 151.7 mm to (202.0, 36.5), turned to 180 degrees
- moved U3 136.1 mm to (175.5, 47.1), turned to 180 degrees
- moved SW1 128.3 mm to (190.6, 49.5)
- moved J3 127.9 mm to (173.8, 61.0), turned to 180 degrees
- moved J4 124.4 mm to (177.4, 61.0)
- moved C3 109.0 mm to (157.7, 62.8), turned to 180 degrees
- moved SW2 104.4 mm to (129.9, 34.6), turned to -90 degrees
- moved U5 103.4 mm to (138.9, 44.1), turned to 180 degrees
- moved C1 99.6 mm to (157.6, 67.6), turned to 180 degrees
- moved U2 96.2 mm to (157.7, 58.0), turned to 180 degrees
- moved R1 95.8 mm to (157.0, 51.3)
- moved C4 95.6 mm to (146.1, 65.0)
- moved R2 95.6 mm to (156.9, 53.5)
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Connections:
- SW2 pad 1: unconnected-(SW2-Pad1) -> GND
- SW2 pad 2: GND -> Net-(U1-GPIO0)
- U1 pad 0: unconnected-(U1-GPIO0-Pad0) -> Net-(U1-GPIO0)
- U1 pad 1: unconnected-(U1-GPIO1-Pad1) -> Net-(J14-Pin_3)
- U1 pad 10: unconnected-(U1-GPIO10-Pad10) -> INB1
- U1 pad 20: unconnected-(U1-GPIO20-Pad20) -> INB2
- U1 pad 21: unconnected-(U1-GPIO21-Pad21) -> PWMB
- U1 pad 3: unconnected-(U1-GPIO3-Pad3) -> QTR_DER
- U1 pad 4: unconnected-(U1-GPIO4-Pad4) -> QTR_IZQ
- U1 pad 5: unconnected-(U1-GPIO5-Pad5) -> PWMA
- U1 pad 6: unconnected-(U1-GPIO6-Pad6) -> INA2
- U1 pad 7: unconnected-(U1-GPIO7-Pad7) -> INA1
- U1 pad 8: unconnected-(U1-GPIO8-Pad8) -> SDA
- U1 pad 9: unconnected-(U1-GPIO9-Pad9) -> SCL
- U3 pad 10: unconnected-(U3-PWMB-Pad10) -> PWMB
- U3 pad 11: unconnected-(U3-BI2-Pad11) -> INB2
- U3 pad 12: unconnected-(U3-BI1-Pad12) -> INB1
- U3 pad 13: Net-(J5-Pin_2) -> +3.3V
- U3 pad 14: unconnected-(U3-AI1-Pad14) -> INA1
- U3 pad 15: unconnected-(U3-AI2-Pad15) -> INA2
- U3 pad 16: unconnected-(U3-PWMA-Pad16) -> PWMA
- U4 pad 10: unconnected-(U4-P5-Pad10) -> VL53_5
- U4 pad 4: unconnected-(U4-P0-Pad4) -> VL53_0
- U4 pad 5: unconnected-(U4-P1-Pad5) -> VL53_1
- U4 pad 6: unconnected-(U4-P2-Pad6) -> VL53_2
- U4 pad 7: unconnected-(U4-P3-Pad7) -> VL53_3
- U4 pad 9: unconnected-(U4-P4-Pad9) -> VL53_4
- U5 pad HV3: unconnected-(U5-PadHV3) -> Net-(J6-Pin_3)
- U5 pad HV4: unconnected-(U5-PadHV4) -> Net-(J7-Pin_3)
- U5 pad LV3: unconnected-(U5-PadLV3) -> QTR_IZQ
- U5 pad LV4: unconnected-(U5-PadLV4) -> QTR_DER
Routing:
- net GND: track 0.00 -> 192.0 mm
- net +3.3V: track 0.00 -> 102.9 mm, vias 0 -> 1
- net SDA: track 0.00 -> 75.1 mm
- net SCL: track 0.10 -> 63.5 mm
- net +5V: track 0.00 -> 60.3 mm
- net VMOT: track 0.00 -> 54.3 mm
- net Net-(U1-GPIO0): track 0.00 -> 47.1 mm
- net Net-(J3-Pin_2): track 0.00 -> 27.4 mm
- net Net-(J3-Pin_1): track 0.00 -> 23.3 mm
- net Net-(J14-Pin_3): track 0.00 -> 23.2 mm
- net Net-(J4-Pin_1): track 0.00 -> 18.9 mm
- net VL53_0: track 0.00 -> 15.6 mm
- net Net-(J4-Pin_2): track 0.00 -> 14.9 mm
- net VL53_3: track 0.00 -> 13.5 mm
- net VL53_1: track 0.00 -> 12.7 mm
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Other:
- board outline added: 96 x 61 mm

Commit message: m,
jkgh
Parts:
- removed C4: 220uf / 25v, Capacitor_THT:CP_Radial_D8.0mm_P3.80mm
- removed R1, R2: 10k, Resistor_SMD:R_0805_2012Metric_Pad1.20x1.40mm_HandSolder
- removed U5: LEVEL-SHIFTER-4ch, BOB-12009:CONV_BOB-12009
- added C5: 220uf / 25v, Capacitor_THT:CP_Radial_D6.3mm_P2.50mm, F.Cu at (169.9, 106.2)
- added J5: Conn_01x04_Pin, Connector_PinHeader_2.54mm:PinHeader_1x04_P2.54mm_Vertical, F.Cu at (179.8, 96.7)
- added SW3: SW_Push, Button_Switch_THT:SW_PUSH_6mm_H4.3mm, F.Cu at (156.5, 103.4)
- J10, J11, J12, J13, J8, J9: value Conn_01x05_Pin -> Conn_01x04_Pin; footprint Connector_PinHeader_2.54mm:PinHeader_1x05_P2.54mm_Vertical -> Connector_PinHeader_2.54mm:PinHeader_1x04_P2.54mm_Vertical
- U4: value PCF8574AT -> BOB-12009; footprint Package_SO:SOIC-16W_7.5x10.3mm_P1.27mm -> BOB-12009:CONV_BOB-12009; moved to F.Cu
- moved J7 83.9 mm to (163.3, 108.6), turned to 180 degrees
- moved J14 83.6 mm to (185.6, 106.6), turned to 180 degrees
- moved J6 82.1 mm to (159.8, 108.7), turned to 180 degrees
- moved J11 75.8 mm to (165.4, 96.7), turned to 180 degrees
- moved J10 75.5 mm to (169.0, 96.7), turned to 180 degrees
- moved J9 75.2 mm to (172.6, 96.7), turned to 180 degrees
- moved J8 75.0 mm to (176.2, 96.7), turned to 180 degrees
- moved J13 73.6 mm to (158.2, 96.7), turned to 180 degrees
- moved J12 72.9 mm to (161.8, 96.7), turned to 180 degrees
- moved SW1 70.0 mm to (226.9, 109.3), turned to 90 degrees
- moved D1 65.2 mm to (223.1, 101.0), turned to 0 degrees
- moved SW2 63.7 mm to (154.9, 93.2)
- moved U1 63.4 mm to (190.9, 99.1)
- moved J1 63.0 mm to (229.6, 93.1), turned to -90 degrees
- moved U4 62.9 mm to (173.3, 105.1), turned to -90 degrees
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Connections:
- U1 pad 1: Net-(J14-Pin_3) -> Net-(U1-GPIO1)
- U1 pad 2: unconnected-(U1-GPIO2-Pad2) -> Net-(J14-Pin_3)
- U3 pad 4: Net-(J4-Pin_2) -> Net-(J4-Pin_1)
- U3 pad 5: Net-(J4-Pin_1) -> Net-(J4-Pin_2)
Routing:
- net Net-(U1-GPIO1): track 0.00 -> 64.3 mm, vias 0 -> 1
- net SDA: track 75.1 -> 52.2 mm
- net +5V: track 60.3 -> 43.2 mm
- net Net-(J14-Pin_3): track 23.2 -> 6.95 mm
- net VL53_0: track 15.6 -> 0.00 mm
- net Net-(J6-Pin_3): track 9.58 -> 24.5 mm
- net VMOT: track 54.3 -> 39.9 mm
- net VL53_3: track 13.5 -> 0.00 mm
- net SCL: track 63.5 -> 50.6 mm
- net VL53_1: track 12.7 -> 0.00 mm
- net VL53_2: track 12.5 -> 0.00 mm
- net VL53_5: track 12.4 -> 0.00 mm
- net VL53_4: track 12.1 -> 0.00 mm
- net Net-(J7-Pin_3): track 5.09 -> 17.0 mm
- net GND: track 192.0 -> 181.0 mm
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Other:
- board outline removed

Commit message: modelo 3d del pcb en el diseño
agregue al diseño del minisumo  el modelo 3d de la pcb
Other:
- board outline added: 90.4 x 29.1 mm
