File: HardWare/V2_robot_controller/V2_robot_controller/V2_robot_controller.kicad_pcb (KiCad board)
At the start: 2 copper layers, 96 x 61 mm, 34 parts, among them J1 XT30UPB-M, J10 Conn_01x05_Pin, J11 Conn_01x05_Pin, J12 Conn_01x05_Pin, J13 Conn_01x05_Pin, J14 Conn_01x03_Pin, J2 XT30UPB-M, J4 Conn_01x02_Pin, J5 Conn_01x02_Pin, J6 Conn_01x03_Pin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

Commit message: m,
jkgh
Parts:
- moved D1 223.3 mm to (252.8, 112.5), turned to -90 degrees
- moved J1 198.1 mm to (259.9, 120.5), turned to 180 degrees
- moved J2 195.5 mm to (259.9, 114.7)
- moved SW1 187.2 mm to (248.7, 118.7), turned to 90 degrees
- moved U4 151.1 mm to (197.3, 113.4), turned to -90 degrees
- moved U2 149.1 mm to (187.5, 115.9), turned to 90 degrees
- moved C7 127.7 mm to (235.4, 116.8)
- moved C9 127.7 mm to (219.4, 116.6)
- moved C10 127.7 mm to (222.7, 116.2)
- moved C8 127.7 mm to (238.7, 116.5)
- moved J4 127.7 mm to (244.2, 124.9)
- moved J5 127.7 mm to (228.3, 124.7)
- moved R5 127.7 mm to (243.1, 120.4)
- moved U7 127.7 mm to (242.4, 115.1)
- moved U8 127.7 mm to (226.5, 114.9)
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Other:
- outline, holes or cut-outs redrawn
